Commit message: getting slam up using dynamic map

File: src/toulouse_rover/urdf/toulouse.urdf.xacro (robot description, xacro)
@@ -3,9 +3,9 @@
   <link name="base_link">
   </link>
-  <link name="base_laser">
+  <link name="base_footprint">
   </link>
   <joint name="base_laser_to_base_link" type="fixed">
     <parent link="base_link"/>
-    <child link="base_laser"/>
+    <child link="base_footprint"/>
     <origin xyz="0 0 0.25"/>
   </joint>

Commit message: updating config files

File: src/toulouse_rover/urdf/toulouse.urdf.xacro (robot description, xacro)
@@ -5,8 +5,15 @@
   <link name="base_footprint">
   </link>
-  <joint name="base_laser_to_base_link" type="fixed">
+  <joint name="base_lidar_to_base_link" type="fixed">
     <parent link="base_link"/>
     <child link="base_footprint"/>
     <origin xyz="0 0 0.25"/>
   </joint>
+  <link name="laser_frame">
+  </link>
+  <joint name="base_laser_to_base_link" type="fixed">
+    <parent link="base_footprint"/>
+    <child link="laser_frame"/>
+    <origin xyz="0 0 0.2"/>
+  </joint>
 </robot>

Commit message: updating to do mapping

File: src/toulouse_rover/urdf/toulouse.urdf.xacro (robot description, xacro)
@@ -5,5 +5,5 @@
   <link name="base_footprint">
   </link>
-  <joint name="base_lidar_to_base_link" type="fixed">
+  <joint name="base_footprint_to_base_link" type="fixed">
     <parent link="base_link"/>
     <child link="base_footprint"/>
@@ -15,5 +15,5 @@
     <parent link="base_footprint"/>
     <child link="laser_frame"/>
-    <origin xyz="0 0 0.2"/>
+    <origin xyz="0 0 0.2" rpy="0 0 3.1416"/>
   </joint>
 </robot>
